File: KiCad/VecCRT_lightgun.kicad_pcb (KiCad board)
At the start: 2 copper layers, 50 x 30 mm, 11 parts, among them J8 Conn_01x03, K1 SchEin, Q7 2N7000, U1 555, X1 OPL820-OC

Commit message: small fixes
Parts:
- D1, K1: footprint RG:PSS_2W -> RG:Pins_2
- J8, X1: footprint RG:PSS_3W -> RG:Pins_3
- moved X1 33.3 mm to (8.89, 22.9), turned to 90 degrees
- moved J8 33.1 mm to (41.9, 20.3)
- moved D1 0.27 mm to (41.9, 8.89), turned to 90 degrees
- turned K1 to -90 degrees
Connections:
- J8 pad 1: /5V -> GND
- J8 pad 3: GND -> /5V
Routing:
- net Net-(Q7-PadG): track 47.3 -> 20.3 mm
- net Net-(J8-Pad2): track 15.2 -> 35.1 mm
- net GND: track 39.6 -> 40.6 mm
- net /5V: track 131.9 -> 132.6 mm
