File: KiCad/VecCRTtap.kicad_sch (KiCad schematic)
At the start: 34 parts, among them J1 X, J2 Conn_02x08_Odd_Even, J3 Y, J4 Conn_02x08_Odd_Even, J5 Z, J6 Conn_01x03, J7 Conn_01x03, K1 1UM, Q1 BS250, Q2 BS170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

Commit message: small fixes
Parts:
- J6, J7: footprint RG:PSS_3 -> RG:PSS_3W
Connections:
- net GND: now also RV1.1, RV2.1; no longer RV1.3, RV2.3
- net Xout: now also RV1.3; no longer RV1.1
- net Yout: now also RV2.3; no longer RV2.1
Changed lines of the file:
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@@
     (property "Reference" "J6" (id 0) (at 34.29 104.14 0))
     (property "Value" "Conn_01x03" (id 1) (at 34.29 114.3 0))
-    (property "Footprint" "RG:PSS_3" (id 2) (at 34.29 109.22 0)
+    (property "Footprint" "RG:PSS_3W" (id 2) (at 34.29 109.22 0)
       (effects (font (size 1.27 1.27)) hide)
     )
@@
     (pin "2")
   )
-  (symbol (lib_id "Device:R_Potentiometer") (at 80.01 26.035 0) (unit 1)
+  (symbol (lib_id "Device:R_Potentiometer") (at 80.01 26.035 0) (mirror x) (unit 1)
     (in_bom yes) (on_board yes)
     (property "Reference" "RV1" (id 0) (at 75.565 26.035 90))
@@
     (property "Reference" "J7" (id 0) (at 54.61 104.14 0))
     (property "Value" "Conn_01x03" (id 1) (at 54.61 114.3 0))
-    (property "Footprint" "RG:PSS_3" (id 2) (at 54.61 109.22 0)
+    (property "Footprint" "RG:PSS_3W" (id 2) (at 54.61 109.22 0)
       (effects (font (size 1.27 1.27)) hide)
     )
@@
     (pin "1")
   )
-  (symbol (lib_id "Device:R_Potentiometer") (at 80.01 50.8 0) (unit 1)
+  (symbol (lib_id "Device:R_Potentiometer") (at 80.01 50.8 0) (mirror x) (unit 1)
     (in_bom yes) (on_board yes)
     (property "Reference" "RV2" (id 0) (at 75.565 50.8 90))
@@
     )
     (path "/113af575-d8af-4171-aeaa-caf7c2cedc92"
-      (reference "J6") (unit 1) (value "Conn_01x03") (footprint "RG:PSS_3")
+      (reference "J6") (unit 1) (value "Conn_01x03") (footprint "RG:PSS_3W")
     )
     (path "/8a9d1136-9fbc-401a-9c95-0d79467eb8bd"
-      (reference "J7") (unit 1) (value "Conn_01x03") (footprint "RG:PSS_3")
+      (reference "J7") (unit 1) (value "Conn_01x03") (footprint "RG:PSS_3W")
     )
     (path "/3e4fccb9-351f-484d-bbb9-17d684151a82"
