File: KiCad/VecCRT.kicad_sch (KiCad schematic)
At the start: 106 parts, among them J1 RaspiGPIO40, J2 Conn_02x08_Odd_Even, J3 Conn_01x04_Female, Q1 2N7000, Q10 BSS138, Q11 BSS138, Q12 BSS138, Q13 2N7000, Q14 BSS138, Q2 2N7000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

Commit message: kicad fixes
Parts:
- removed D2: 1N914, Diode_THT:D_DO-35_SOD27_P7.62mm_Horizontal, symbol Diode:1N914
- added C13: 100n, RG:SM-1206B, symbol Device:C
- added D2: BAT42, Diode_THT:D_DO-35_SOD27_P7.62mm_Horizontal, symbol Diode:BAT42
- added R26: 680k, RG:R4-2, symbol Device:R
Connections:
- net +5V: now also D2.1 (K)
- net GND: now also C13.2
- net at C5.2, R21.1, U4.13: now also D2.2 (A), R26.1
- net at R21.2, RV2.3: now also R26.2
- net at JP3.3 (B), U9.Vo: now also C13.1
Other:
- note added: "C1 and C3: select for equality"
- moved on the sheet: U4F, U9

Commit message: Fixes in Schematics
Parts:
- C13: value 100n -> 2.2u
- R25: value 6.8k -> 3.9k
- R26: footprint RG:R4-2 -> RG:SM-1206B
Connections:
- net -5V: now also J2.16 (Pin_16)
- no-connect marks 11 -> 10
Changed lines of the file:
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@@
     (title "Vector Drawing for WWI")
     (date "2023-09-08")
-    (rev "1.0d")
+    (rev "1.0e")
   )
   (junction (at 62.23 26.67) (diameter 0) (color 0 0 0 0)
@@
   )
   (no_connect (at 59.69 54.61))
-  (no_connect (at 278.13 128.27))
   (no_connect (at 59.69 19.05))
   (no_connect (at 21.59 54.61))
@@
     (stroke (width 0) (type default) (color 0 0 0 0))
   )
+  (wire (pts (xy 278.13 128.27) (xy 283.845 128.27))
+    (stroke (width 0) (type default) (color 0 0 0 0))
+  )
   (wire (pts (xy 281.94 166.37) (xy 281.94 177.8))
     (stroke (width 0) (type default) (color 0 0 0 0))
@@
     (in_bom yes) (on_board yes)
     (property "Reference" "R25" (id 0) (at 99.568 96.52 90))
-    (property "Value" "6.8k" (id 1) (at 101.6 96.52 90))
+    (property "Value" "3.9k" (id 1) (at 101.6 96.52 90))
     (property "Footprint" "RG:R4-2" (id 2) (at 103.378 96.52 90)
       (effects (font (size 1.27 1.27)) hide)
@@
     (pin "2")
   )
+  (symbol (lib_id "power:-5V") (at 283.845 128.27 270) (unit 1)
+    (in_bom yes) (on_board yes)
+    (property "Reference" "#PWR0101" (id 0) (at 286.385 128.27 0)
+      (effects (font (size 1.27 1.27)) hide)
+    )
+    (property "Value" "-5V" (id 1) (at 287.655 128.27 0))
+    (property "Footprint" "" (id 2) (at 283.845 128.27 0)
+      (effects (font (size 1.27 1.27)) hide)
+    )
+    (property "Datasheet" "" (id 3) (at 283.845 128.27 0)
+      (effects (font (size 1.27 1.27)) hide)
+    )
+    (pin "1")
+  )
   (symbol (lib_id "rg:4011") (at 46.99 138.43 0) (unit 4)
     (in_bom yes) (on_board yes)
@@
     (property "Reference" "R26" (id 0) (at 128.143 96.52 90))
     (property "Value" "680k" (id 1) (at 130.175 96.52 90))
-    (property "Footprint" "RG:R4-2" (id 2) (at 131.953 96.52 90)
+    (property "Footprint" "RG:SM-1206B" (id 2) (at 131.953 96.52 90)
       (effects (font (size 1.27 1.27)) hide)
     )
@@
       (effects (font (size 1.27 1.27)) (justify left))
     )
-    (property "Value" "100n" (id 1) (at 128.905 186.69 0)
+    (property "Value" "2.2u" (id 1) (at 128.905 186.69 0)
       (effects (font (size 1.27 1.27)) (justify left))
     )
@@
       (reference "#PWR046") (unit 1) (value "GND") (footprint "")
     )
+    (path "/7ae8993a-49e8-4236-aab7-063996a47c7c"
+      (reference "#PWR0101") (unit 1) (value "-5V") (footprint "")
+    )
     (path "/00000000-0000-0000-0000-00006452fc22"
       (reference "C1") (unit 1) (value "10n") (footprint "RG:C2-2")
@@
     )
     (path "/df36c596-67fa-45c2-996a-ec8d82c4adfb"
-      (reference "C13") (unit 1) (value "100n") (footprint "RG:SM-1206B")
+      (reference "C13") (unit 1) (value "2.2u") (footprint "RG:SM-1206B")
     )
     (path "/00000000-0000-0000-0000-000064793672"
@@
     )
     (path "/00000000-0000-0000-0000-000064830a2d"
-      (reference "R25") (unit 1) (value "6.8k") (footprint "RG:R4-2")
+      (reference "R25") (unit 1) (value "3.9k") (footprint "RG:R4-2")
     )
     (path "/d8fab9e3-9396-4d97-abd9-dd8b0ec5fe18"
-      (reference "R26") (unit 1) (value "680k") (footprint "RG:R4-2")
+      (reference "R26") (unit 1) (value "680k") (footprint "RG:SM-1206B")
     )
     (path "/00000000-0000-0000-0000-000064a6090c"
