File: KiCad/VecCRT.kicad_sch (KiCad schematic)
At the start: 108 parts, among them J1 RaspiGPIO40, J2 Conn_02x08_Odd_Even, J3 Conn_01x04_Female, Q1 2N7000, Q10 BSS138, Q11 BSS138, Q12 BSS138, Q13 2N7000, Q14 BSS138, Q2 2N7000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

Commit message: Fix symbol reference to local library
Parts:
- J1: footprint RG:Wannenstecker_2x20_V -> Connector_PinHeader_2.54mm:PinHeader_2x20_P2.54mm_Vertical
- U4: symbol rg:40106 -> Library:40106
Changed lines of the file:
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@@
     (pin "2")
   )
-  (symbol (lib_name "BS170_2") (lib_id "rg:BS170") (at 64.77 96.52 0) (unit 1)
+  (symbol (lib_id "rg:BS170") (at 64.77 96.52 0) (unit 1)
     (in_bom yes) (on_board yes)
     (property "Reference" "Q2" (id 0) (at 65.024 92.202 0)
@@
     (pin "1")
   )
-  (symbol (lib_id "rg:40106") (at 140.335 104.14 0) (unit 6)
+  (symbol (lib_id "Library:40106") (at 140.335 104.14 0) (unit 6)
     (in_bom yes) (on_board yes)
     (property "Reference" "U4" (id 0) (at 138.43 99.06 0)
@@
     (pin "1")
   )
-  (symbol (lib_id "rg:40106") (at 132.08 69.85 0) (unit 2)
+  (symbol (lib_id "Library:40106") (at 132.08 69.85 0) (unit 2)
     (in_bom yes) (on_board yes)
     (property "Reference" "U4" (id 0) (at 130.175 64.77 0)
@@
     (pin "7")
   )
-  (symbol (lib_name "2N7002_3") (lib_id "rg:2N7002") (at 196.85 127 0) (unit 1)
+  (symbol (lib_id "rg:2N7002") (at 196.85 127 0) (unit 1)
     (in_bom yes) (on_board yes)
     (property "Reference" "Q5" (id 0) (at 197.104 122.682 0)
@@
     (pin "1")
   )
-  (symbol (lib_name "2N7002_2") (lib_id "rg:2N7002") (at 196.85 165.1 0) (unit 1)
+  (symbol (lib_id "rg:2N7002") (at 196.85 165.1 0) (unit 1)
     (in_bom yes) (on_board yes)
     (property "Reference" "Q13" (id 0) (at 197.104 160.782 0)
@@
     (pin "S")
   )
-  (symbol (lib_name "BS170_1") (lib_id "rg:BS170") (at 104.14 69.85 0) (unit 1)
+  (symbol (lib_id "rg:BS170") (at 104.14 69.85 0) (unit 1)
     (in_bom yes) (on_board yes)
     (property "Reference" "Q1" (id 0) (at 104.394 65.532 0)
@@
     (pin "S")
   )
-  (symbol (lib_id "rg:40106") (at 116.84 69.85 0) (unit 1)
+  (symbol (lib_id "Library:40106") (at 116.84 69.85 0) (unit 1)
     (in_bom yes) (on_board yes)
     (property "Reference" "U4" (id 0) (at 114.935 64.77 0)
@@
     (property "Reference" "J1" (id 0) (at 29.21 7.62 0))
     (property "Value" "RaspiGPIO40" (id 1) (at 40.64 10.16 0))
-    (property "Footprint" "RG:Wannenstecker_2x20_V" (id 2) (at 40.64 34.925 90)
+    (property "Footprint" "Connector_PinHeader_2.54mm:PinHeader_2x20_P2.54mm_Vertical" (id 2) (at 40.64 34.925 90)
       (effects (font (size 1.27 1.27)) hide)
     )
@@
     (pin "2")
   )
-  (symbol (lib_name "BS170_5") (lib_id "rg:BS170") (at 64.77 138.43 0) (unit 1)
+  (symbol (lib_id "rg:BS170") (at 64.77 138.43 0) (unit 1)
     (in_bom yes) (on_board yes)
     (property "Reference" "Q8" (id 0) (at 65.024 134.112 0)
@@
     (pin "2")
   )
-  (symbol (lib_name "2N7002_1") (lib_id "rg:2N7002") (at 29.21 101.6 0) (unit 1)
+  (symbol (lib_id "rg:2N7002") (at 29.21 101.6 0) (unit 1)
     (in_bom yes) (on_board yes)
     (property "Reference" "Q3" (id 0) (at 29.464 97.282 0)
@@
     )
     (path "/cb656c73-447f-4ef0-8c6c-c591e84dda3b"
-      (reference "J1") (unit 1) (value "RaspiGPIO40") (footprint "RG:Wannenstecker_2x20_V")
+      (reference "J1") (unit 1) (value "RaspiGPIO40") (footprint "Connector_PinHeader_2.54mm:PinHeader_2x20_P2.54mm_Vertical")
     )
     (path "/0cdd7481-1b83-4e49-a89a-ad070f146b13"
